Commit message: Rename custom_robot_sim to chocolate_factory_sim

File: chocolate_factory_sim/urdf/box.urdf.xacro (robot description, xacro)
@@ -1,6 +1,6 @@
 <?xml version="1.0" ?>
 <robot name="box" xmlns:xacro="http://ros.org/wiki/xacro">
-    <xacro:include filename="$(find custom_robot_sim)/urdf/inertial_macros.urdf.xacro" />
-    <xacro:include filename="$(find custom_robot_sim)/urdf/materials.urdf.xacro" />
+    <xacro:include filename="$(find chocolate_factory_sim)/urdf/inertial_macros.urdf.xacro" />
+    <xacro:include filename="$(find chocolate_factory_sim)/urdf/materials.urdf.xacro" />
     <xacro:property name="wall_length" value="0.105" />
     <xacro:property name="wall_width" value="0.005" />

File: chocolate_factory_sim/urdf/cube.urdf.xacro (robot description, xacro)
@@ -1,6 +1,6 @@
 <?xml version="1.0" ?>
 <robot name="cube" xmlns:xacro="http://ros.org/wiki/xacro">
-    <xacro:include filename="$(find custom_robot_sim)/urdf/inertial_macros.urdf.xacro" />
-    <xacro:include filename="$(find custom_robot_sim)/urdf/materials.urdf.xacro" />
+    <xacro:include filename="$(find chocolate_factory_sim)/urdf/inertial_macros.urdf.xacro" />
+    <xacro:include filename="$(find chocolate_factory_sim)/urdf/materials.urdf.xacro" />
     <xacro:property name="size" value="0.05" />
     <link name="cube_link">

File: chocolate_factory_sim/urdf/robot_control.gazebo.xacro (robot description, xacro)
@@ -4,5 +4,5 @@
     <gazebo>
         <plugin filename="gz_ros2_control-system" name="gz_ros2_control::GazeboSimROS2ControlPlugin">
-            <parameters>$(find custom_robot_sim)/config/controller_config.yaml</parameters>
+            <parameters>$(find chocolate_factory_sim)/config/controller_config.yaml</parameters>
         </plugin>
     </gazebo>

File: chocolate_factory_sim/urdf/robot_description.urdf.xacro (robot description, xacro)
@@ -1,7 +1,7 @@
 <?xml version="1.0" ?>
 <robot name="custom_manipulator" xmlns:xacro="http://ros.org/wiki/xacro">
-    <xacro:include filename="$(find custom_robot_sim)/urdf/inertial_macros.urdf.xacro" />
-    <xacro:include filename="$(find custom_robot_sim)/urdf/robot_control.gazebo.xacro" />
-    <xacro:include filename="$(find custom_robot_sim)/urdf/materials.urdf.xacro" />
+    <xacro:include filename="$(find chocolate_factory_sim)/urdf/inertial_macros.urdf.xacro" />
+    <xacro:include filename="$(find chocolate_factory_sim)/urdf/robot_control.gazebo.xacro" />
+    <xacro:include filename="$(find chocolate_factory_sim)/urdf/materials.urdf.xacro" />
     <link name="base_footprint"/>
     <joint name="footprint_joint" type="fixed">
@@ -17,5 +17,5 @@
             <origin xyz="0 0 0" rpy="0 0 0"/>
             <geometry>
-                <mesh filename="$(find custom_robot_sim)/meshes/arm_base_plate.stl" />
+                <mesh filename="$(find chocolate_factory_sim)/meshes/arm_base_plate.stl" />
             </geometry>
             <material name="blue"/>
@@ -52,5 +52,5 @@
             <origin xyz="0 0 0" rpy="0 0 0"/>
             <geometry>
-                <mesh filename="$(find custom_robot_sim)/meshes/arm_base_link.stl" />
+                <mesh filename="$(find chocolate_factory_sim)/meshes/arm_base_link.stl" />
             </geometry>
             <material name="blue"/>
@@ -87,5 +87,5 @@
             <origin xyz="0 -${0.285/2} 0" rpy="${pi/2} 0 0"/>
             <geometry>
-                <mesh filename="$(find custom_robot_sim)/meshes/link_1.stl" />
+                <mesh filename="$(find chocolate_factory_sim)/meshes/link_1.stl" />
             </geometry>
             <material name="blue"/>
@@ -128,5 +128,5 @@
             <origin xyz="0 -${0.27/2} 0" rpy="${pi/2} 0 0"/>
             <geometry>
-                <mesh filename="$(find custom_robot_sim)/meshes/link_2.stl" />
+                <mesh filename="$(find chocolate_factory_sim)/meshes/link_2.stl" />
             </geometry>
             <material name="blue"/>
@@ -157,5 +157,5 @@
             <origin xyz="0 -0.08 0" rpy="${pi/2} 0 0"/>
             <geometry>
-                <mesh filename="$(find custom_robot_sim)/meshes/link_3.stl" />
+                <mesh filename="$(find chocolate_factory_sim)/meshes/link_3.stl" />
             </geometry>
             <material name="blue"/>
@@ -192,5 +192,5 @@
             <origin xyz="0 0 0" rpy="0 0 0"/>
             <geometry>
-                <mesh filename="$(find custom_robot_sim)/meshes/gripper_base.stl" />
+                <mesh filename="$(find chocolate_factory_sim)/meshes/gripper_base.stl" />
             </geometry>
             <material name="blue"/>
@@ -227,5 +227,5 @@
             <origin xyz="0 0 0" rpy="0 -${pi/2} 0"/>
             <geometry>
-                <mesh filename="$(find custom_robot_sim)/meshes/gripper_finger.stl" />
+                <mesh filename="$(find chocolate_factory_sim)/meshes/gripper_finger.stl" />
             </geometry>
             <material name="blue"/>
@@ -263,5 +263,5 @@
             <origin xyz="0 0 0" rpy="0 -${pi/2} 0"/>
             <geometry>
-                <mesh filename="$(find custom_robot_sim)/meshes/gripper_finger.stl" />
+                <mesh filename="$(find chocolate_factory_sim)/meshes/gripper_finger.stl" />
             </geometry>
             <material name="blue"/>

File: chocolate_factory_sim/urdf/robot_description_no_dummy.urdf.xacro (robot description, xacro)
@@ -1,7 +1,7 @@
 <?xml version="1.0" ?>
 <robot name="custom_manipulator" xmlns:xacro="http://ros.org/wiki/xacro">
-    <xacro:include filename="$(find custom_robot_sim)/urdf/inertial_macros.urdf.xacro" />
-    <xacro:include filename="$(find custom_robot_sim)/urdf/robot_control.gazebo.xacro" />
-    <xacro:include filename="$(find custom_robot_sim)/urdf/materials.urdf.xacro" />
+    <xacro:include filename="$(find chocolate_factory_sim)/urdf/inertial_macros.urdf.xacro" />
+    <xacro:include filename="$(find chocolate_factory_sim)/urdf/robot_control.gazebo.xacro" />
+    <xacro:include filename="$(find chocolate_factory_sim)/urdf/materials.urdf.xacro" />
     <!--############################### -->
     <!-- ARM BASE PLATE -->
@@ -11,5 +11,5 @@
             <origin xyz="0 0 0" rpy="0 0 0"/>
             <geometry>
-                <mesh filename="$(find custom_robot_sim)/meshes/arm_base_plate.stl" />
+                <mesh filename="$(find chocolate_factory_sim)/meshes/arm_base_plate.stl" />
             </geometry>
             <material name="blue"/>
@@ -46,5 +46,5 @@
             <origin xyz="0 0 0" rpy="0 0 0"/>
             <geometry>
-                <mesh filename="$(find custom_robot_sim)/meshes/arm_base_link.stl" />
+                <mesh filename="$(find chocolate_factory_sim)/meshes/arm_base_link.stl" />
             </geometry>
             <material name="blue"/>
@@ -81,5 +81,5 @@
             <origin xyz="0 -${0.285/2} 0" rpy="${pi/2} 0 0"/>
             <geometry>
-                <mesh filename="$(find custom_robot_sim)/meshes/link_1.stl" />
+                <mesh filename="$(find chocolate_factory_sim)/meshes/link_1.stl" />
             </geometry>
             <material name="blue"/>
@@ -122,5 +122,5 @@
             <origin xyz="0 -${0.27/2} 0" rpy="${pi/2} 0 0"/>
             <geometry>
-                <mesh filename="$(find custom_robot_sim)/meshes/link_2.stl" />
+                <mesh filename="$(find chocolate_factory_sim)/meshes/link_2.stl" />
             </geometry>
             <material name="blue"/>
@@ -151,5 +151,5 @@
             <origin xyz="0 -0.08 0" rpy="${pi/2} 0 0"/>
             <geometry>
-                <mesh filename="$(find custom_robot_sim)/meshes/link_3.stl" />
+                <mesh filename="$(find chocolate_factory_sim)/meshes/link_3.stl" />
             </geometry>
             <material name="blue"/>
@@ -186,5 +186,5 @@
             <origin xyz="0 0 0" rpy="0 0 0"/>
             <geometry>
-                <mesh filename="$(find custom_robot_sim)/meshes/gripper_base.stl" />
+                <mesh filename="$(find chocolate_factory_sim)/meshes/gripper_base.stl" />
             </geometry>
             <material name="blue"/>
@@ -221,5 +221,5 @@
             <origin xyz="0 0 0" rpy="0 -${pi/2} 0"/>
             <geometry>
-                <mesh filename="$(find custom_robot_sim)/meshes/gripper_finger.stl" />
+                <mesh filename="$(find chocolate_factory_sim)/meshes/gripper_finger.stl" />
             </geometry>
             <material name="blue"/>
@@ -257,5 +257,5 @@
             <origin xyz="0 0 0" rpy="0 -${pi/2} 0"/>
             <geometry>
-                <mesh filename="$(find custom_robot_sim)/meshes/gripper_finger.stl" />
+                <mesh filename="$(find chocolate_factory_sim)/meshes/gripper_finger.stl" />
             </geometry>
             <material name="blue"/>

File: chocolate_factory_sim/urdf/robot_stand.urdf.xacro (robot description, xacro)
@@ -1,5 +1,5 @@
 <?xml version="1.0" ?>
 <robot name="robot_stand" xmlns:xacro="http://ros.org/wiki/xacro">
-    <xacro:include filename="$(find custom_robot_sim)/urdf/robot_description_no_dummy.urdf.xacro" />
+    <xacro:include filename="$(find chocolate_factory_sim)/urdf/robot_description_no_dummy.urdf.xacro" />
     <link name="base_footprint"/>
     <joint name="footprint_joint" type="fixed">

File: chocolate_factory_sim/urdf/table.urdf.xacro (robot description, xacro)
@@ -1,6 +1,6 @@
 <?xml version="1.0" ?>
 <robot name="table" xmlns:xacro="http://ros.org/wiki/xacro">
-    <xacro:include filename="$(find custom_robot_sim)/urdf/inertial_macros.urdf.xacro" />
-    <xacro:include filename="$(find custom_robot_sim)/urdf/materials.urdf.xacro" />
+    <xacro:include filename="$(find chocolate_factory_sim)/urdf/inertial_macros.urdf.xacro" />
+    <xacro:include filename="$(find chocolate_factory_sim)/urdf/materials.urdf.xacro" />
     <xacro:macro name="table_leg" params="link_name">
         <link name="${link_name}">
