Commit message: Update joint types and parameters in URDF
Changed joint types from 'continuous' to 'revolute' and updated limits and initial values for several joints.

File: chocolate_robot_description/urdf/chocolate_robot_gazebo.urdf (robot description, URDF)
Before this commit: robot chocolate_robot, 7 links, 6 joints
Joints:
- joint joint_1: limit effort=100.0 velocity=1.00 -> lower=-3.141593 upper=3.141593 effort=100 velocity=100; type continuous -> revolute
- joint joint_2: axis 0.000000 0.000000 1.000000 -> 0.000000 0.000000 -1.000000; limit effort=100.0 velocity=1.00 -> lower=-3.141593 upper=3.141593 effort=100 velocity=100; origin xyz=0.000000 0.101002 -0.204715 rpy=1.570796 0.000000 0.000000 -> xyz=0.000000 0.101002 -0.204715 rpy=1.570796 -0.698132 0.000000; type continuous -> revolute
- joint joint_3: limit effort=100.0 velocity=1.00 -> lower=-3.141593 upper=3.141593 effort=100 velocity=100; type continuous -> revolute
- joint joint_4: axis 0.000000 0.000000 1.000000 -> 0.000000 0.000000 -1.000000; limit effort=100.0 velocity=1.00 -> lower=-3.141593 upper=3.141593 effort=100 velocity=100; origin xyz=0.515241 0.432339 0.000012 rpy=-3.141593 0.000000 0.000000 -> xyz=0.515241 0.432339 0.000012 rpy=-3.141593 0.000000 0.698132; type continuous -> revolute
- joint joint_5: limit effort=100.0 velocity=1.00 -> lower=-3.141593 upper=3.141593 effort=100 velocity=100; type continuous -> revolute
